File: Electronics/cube-connector.sch (EAGLE design)
At the start: 4 parts

Commit message: File organising...
Parts:
- removed GND, SCL, SDA, V+: (no value), pinhead:PINHD-1X1
Connections:
- removed net GND: GND.1
- removed net SCL: SCL.1
- removed net SDA: SDA.1
- removed net V+: V+.1
Changed lines of the file:
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@@
 </classes>
 <parts>
-<part name="V+" library="pinhead" deviceset="PINHD-1X1" device=""/>
-<part name="GND" library="pinhead" deviceset="PINHD-1X1" device=""/>
-<part name="SDA" library="pinhead" deviceset="PINHD-1X1" device=""/>
-<part name="SCL" library="pinhead" deviceset="PINHD-1X1" device=""/>
 <part name="P+1" library="supply1" deviceset="V+" device=""/>
 <part name="GND1" library="supply1" deviceset="GND" device=""/>
@@
 </plain>
 <instances>
-<instance part="V+" gate="G$1" x="55.88" y="68.58"/>
-<instance part="GND" gate="G$1" x="55.88" y="58.42"/>
-<instance part="SDA" gate="G$1" x="55.88" y="48.26"/>
-<instance part="SCL" gate="G$1" x="55.88" y="38.1"/>
 <instance part="P+1" gate="1" x="38.1" y="76.2"/>
 <instance part="GND1" gate="1" x="38.1" y="53.34"/>
@@
 <net name="V+" class="0">
 <segment>
-<pinref part="V+" gate="G$1" pin="1"/>
 <wire x1="53.34" y1="68.58" x2="38.1" y2="68.58" width="0.1524" layer="91"/>
 <pinref part="P+1" gate="1" pin="V+"/>
@@
 <net name="GND" class="0">
 <segment>
-<pinref part="GND" gate="G$1" pin="1"/>
 <wire x1="53.34" y1="58.42" x2="38.1" y2="58.42" width="0.1524" layer="91"/>
 <pinref part="GND1" gate="1" pin="GND"/>
@@
 <net name="SDA" class="0">
 <segment>
-<pinref part="SDA" gate="G$1" pin="1"/>
 <wire x1="53.34" y1="48.26" x2="27.94" y2="48.26" width="0.1524" layer="91"/>
 <label x="27.94" y="48.26" size="1.778" layer="95"/>
@@
 <net name="SCL" class="0">
 <segment>
-<pinref part="SCL" gate="G$1" pin="1"/>
 <wire x1="53.34" y1="38.1" x2="27.94" y2="38.1" width="0.1524" layer="91"/>
 <label x="27.94" y="38.1" size="1.778" layer="95"/>
